File: SmolISP.kicad_pcb (KiCad board)
At the start: 4 copper layers, 42.2 x 20.3 mm, 31 parts, among them J1 USB_B_Micro, J2 SWD, U1 STM32F103C8Tx, U2 AMS1117-3.3, U3 ATtiny85-20PU, Y1 8 MHz

Commit message: Changes after PCB review
Parts:
- added R1: 10k, Resistor_SMD:R_0805_2012Metric_Pad1.20x1.40mm_HandSolder, F.Cu at (138.4, 113.9)
- U1: value STM32F103C8Tx -> STM32F103C6Tx
- Y1: footprint Crystal:Crystal_SMD_5032-2Pin_5.0x3.2mm -> Crystal:Crystal_SMD_5032-4Pin_5.0x3.2mm
- moved C5 1.77 mm to (151.8, 100.8), turned to 180 degrees
- moved R3 1.23 mm to (164.0, 101.4), turned to 90 degrees
- moved R9 1.09 mm to (136.0, 113.9)
- moved R7 0.38 mm to (137.5, 110.0)
- moved C9 0.18 mm to (151.1, 98.2)
Connections:
- net ISP_AUX_CLOCK renamed EXT_CLOCK
- J1 pad 4: Net-(J1-Pad4) -> (no net)
- U1 pad 1: Net-(U1-Pad1) -> (no net)
- U1 pad 10: Net-(U1-Pad10) -> (no net)
- U1 pad 12: Net-(U1-Pad12) -> (no net)
- U1 pad 13: Net-(U1-Pad13) -> (no net)
- U1 pad 14: Net-(U1-Pad14) -> (no net)
- U1 pad 18: Net-(U1-Pad18) -> (no net)
- U1 pad 19: Net-(U1-Pad19) -> (no net)
- U1 pad 2: Net-(U1-Pad2) -> (no net)
- U1 pad 21: Net-(U1-Pad21) -> (no net)
- U1 pad 22: Net-(U1-Pad22) -> (no net)
- U1 pad 25: Net-(U1-Pad25) -> (no net)
- U1 pad 26: Net-(U1-Pad26) -> (no net)
- U1 pad 27: Net-(U1-Pad27) -> (no net)
- U1 pad 28: Net-(U1-Pad28) -> (no net)
- U1 pad 3: Net-(U1-Pad3) -> (no net)
- U1 pad 30: Net-(U1-Pad30) -> (no net)
- U1 pad 38: Net-(U1-Pad38) -> (no net)
- U1 pad 39: Net-(U1-Pad39) -> (no net)
- U1 pad 4: Net-(U1-Pad4) -> (no net)
- U1 pad 40: Net-(U1-Pad40) -> (no net)
- U1 pad 41: Net-(U1-Pad41) -> (no net)
- U1 pad 42: Net-(U1-Pad42) -> (no net)
- U1 pad 43: Net-(U1-Pad43) -> (no net)
- U1 pad 44: GND -> Net-(R1-Pad2)
- U1 pad 45: Net-(U1-Pad45) -> (no net)
- U1 pad 46: Net-(U1-Pad46) -> (no net)
- U3 pad 3: Net-(U3-Pad3) -> (no net)
- Y1 pad 2: Net-(C2-Pad1) -> GND
Routing:
- net Net-(R1-Pad2): track 0.00 -> 26.5 mm, vias 0 -> 2
- net GND: track 45.2 -> 58.5 mm, vias 24 -> 22
- net Net-(C2-Pad1): track 10.9 -> 12.4 mm
- net Net-(D1-Pad2): track 3.09 -> 2.19 mm
- net ISP_CLK: track 16.7 -> 17.4 mm
- net +3V3: track 50.5 -> 51.1 mm, vias 10 -> 13
Other:
- board text added: "https://github.com/tibordp/SmolISP"
