File: shiny-avr.sch (KiCad schematic (older format))
At the start: 32 parts, among them J1 USB_B_Micro, J2 SWD, U1 STM32F103C6Tx, U2 AMS1117-3.3, U3 ATtiny85-20PU, Y1 8 MHz

Commit message: Relicense + rename
Parts:
- renumbered C7 to C1, C1 to C10, C2 to C11, C8 to C2, C9 to C3, C10 to C4, C3 to C5, C4 to C6, C11 to C7, C5 to C8, C6 to C9, R9 to R1, R3 to R10, R12 to R11, R8 to R12, R7 to R2, R5 to R3, R6 to R4, R4 to R5, R1 to R6, R10 to R7, R2 to R8, R11 to R9, U2 to U1, U1 to U2

Commit message: Add support for ATtiny24/44/48 (#2)
* feat: Add support for ATtinyx4

* fix

Co-authored-by: Tibor Djurica Potpara <tibor.djurica@reddit.com>
Parts:
- added C13: 100n, Capacitor_SMD:C_0805_2012Metric_Pad1.18x1.45mm_HandSolder, symbol Device:C
- added R13, R14, R15, R16: 1k, Resistor_SMD:R_0805_2012Metric_Pad1.20x1.40mm_HandSolder, symbol Device:R
- added R17: 10k, Resistor_SMD:R_0805_2012Metric_Pad1.20x1.40mm_HandSolder, symbol Device:R
- added U4: ATtiny85-20PU, Package_DIP:DIP-14_W7.62mm, symbol MCU_Microchip_ATtiny:ATtiny84-20PU
Connections:
- net +3V3: now also C13.2, R17.1, U4.1 (VCC)
- net EXT_CLOCK: now also R16.1
- net GND: now also C13.1, U4.14 (GND)
- net ISP_CLK: now also R13.1
- net ISP_MISO: now also R14.1
- net ISP_MOSI: now also R15.1
- net ISP_RESET: now also R17.2, U4.4 (~RESET~/PB3)
- new net: R16.2, U4.2 (XTAL1/PB0)
- new net: R15.2, U4.6 (PA7)
- new net: R14.2, U4.8 (PA5)
- new net: R13.2, U4.9 (PA4)
- no-connect marks 29 -> 36
Other:
- note added: "Target ATTINYx4"
- moved on the sheet: C1, C10, C11, C12, C2, C3, C4, C5, C6, C7, C8, C9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
